File: CITADEL/CITADEL 2026/CITADEL 2026.kicad_pcb (KiCad board)
At the start: 2 copper layers, 141.5 x 109.7 mm, 46 parts, among them Q7 SSM3K329R_LF, U3 TJA1051T-3, U4 ESP32-S3-DEVKITC-1-N8R8

Commit message: Added ASTRA logo
Parts:
- added G***: LOGO, LOGO, F.Cu at (99.6, 41.2)
Other:
- board text added: "Jayse Hughes"
- board text added: "PS3"
- board text added: "UAH SHC ASTRA CITADEL V1 1/25/26"
