File: CITADEL/CITADEL 2026/CITADEL 2026.kicad_pcb (KiCad board)
At the start: 2 copper layers, 141.5 x 109.7 mm, 60 parts, among them Q7 SSM3K329R_LF, U1 PCA9685PW_118, U3 TJA1051T-3, U4 ESP32-S3-DEVKITC-1-N8R8

Commit message: Updated Vias
Routing:
- net GND: vias 996 -> 1015
